Commit message: Update ../assets/urdf/vine.urdf

File: assets/urdf/vine.urdf (robot description, URDF)
Before this commit: robot vine_robot, 7 links, 6 joints
Links:
- link base_link: geometry collision cylinder length=0.1 radius=0.025; visual cylinder length=0.1 radius=0.025
- link link_0: geometry collision cylinder length=0.1 radius=0.025; visual cylinder length=0.1 radius=0.025
- link link_1: geometry collision cylinder length=0.1 radius=0.025; visual cylinder length=0.1 radius=0.025
- link link_2: geometry collision cylinder length=0.1 radius=0.025; visual cylinder length=0.1 radius=0.025
Joints:
- joint prismatic_joint_0: limit lower=0.0 upper=0.5 effort=200 velocity=0.2 -> lower=0.0 upper=0.5 effort=200 velocity=0.1
- joint prismatic_joint_1: limit lower=0.0 upper=0.5 effort=200 velocity=0.2 -> lower=0.0 upper=0.5 effort=200 velocity=0.1
- joint prismatic_joint_2: limit lower=0.0 upper=0.5 effort=200 velocity=0.2 -> lower=0.0 upper=0.5 effort=200 velocity=0.1
- joint revolute_joint_1: limit lower=-0.524 upper=0.524 effort=10 velocity=3 -> lower=-0.5236 upper=0.5236 effort=10 velocity=3
- joint revolute_joint_2: limit lower=-0.524 upper=0.524 effort=10 velocity=3 -> lower=-0.5236 upper=0.5236 effort=10 velocity=3

Commit message: Fix big issue with transitions between links and index out of bounds errors

File: assets/urdf/vine.urdf (robot description, URDF)
Before this commit: robot vine_robot, 7 links, 6 joints
Joints:
- joint prismatic_joint_0: limit lower=0.0 upper=0.5 effort=200 velocity=0.1 -> lower=0.0 upper=0.5 effort=200 velocity=1
- joint prismatic_joint_1: limit lower=0.0 upper=0.5 effort=200 velocity=0.1 -> lower=0.0 upper=0.5 effort=200 velocity=1
- joint prismatic_joint_2: limit lower=0.0 upper=0.5 effort=200 velocity=0.1 -> lower=0.0 upper=0.5 effort=200 velocity=1

Commit message: Add joint specific stiffness/damping terms, and increase max joint effort

File: assets/urdf/vine.urdf (robot description, URDF)
Before this commit: robot vine_robot, 7 links, 6 joints
Joints:
- joint prismatic_joint_0: limit lower=0.0 upper=0.5 effort=200 velocity=1 -> lower=0.0 upper=0.5 effort=10000 velocity=1
- joint prismatic_joint_1: limit lower=0.0 upper=0.5 effort=200 velocity=1 -> lower=0.0 upper=0.5 effort=10000 velocity=1
- joint prismatic_joint_2: limit lower=0.0 upper=0.5 effort=200 velocity=1 -> lower=0.0 upper=0.5 effort=10000 velocity=1
- joint revolute_joint_0: limit lower=-3.146 upper=3.146 effort=10 velocity=3 -> lower=-3.146 upper=3.146 effort=10000 velocity=3
- joint revolute_joint_1: limit lower=-0.5236 upper=0.5236 effort=10 velocity=3 -> lower=-0.5236 upper=0.5236 effort=10000 velocity=3
- joint revolute_joint_2: limit lower=-0.5236 upper=0.5236 effort=10 velocity=3 -> lower=-0.5236 upper=0.5236 effort=10000 velocity=3

Commit message: Try to add more links and try to make it work

File: assets/urdf/vine.urdf (robot description, URDF)
Before this commit: robot vine_robot, 7 links, 6 joints
Links:
- added link link_3, mass 0.1; collision cylinder length=0.1 radius=0.025; visual cylinder length=0.1 radius=0.025
- added link link_4, mass 0.1; collision cylinder length=0.1 radius=0.025; visual cylinder length=0.1 radius=0.025
- added link link_5, mass 0.1; collision cylinder length=0.1 radius=0.025; visual cylinder length=0.1 radius=0.025
- added link virtual_link_2
- added link virtual_link_3
- added link virtual_link_4
Joints:
- added joint prismatic_joint_3: type prismatic, parent virtual_link_2, child link_3, origin xyz=0.0 0.0 0.0 rpy=0.0 0.0 0.0, axis 1.0 0.0 0.0, limit lower=0.0 upper=0.5 effort=10000 velocity=1
- added joint prismatic_joint_4: type prismatic, parent virtual_link_3, child link_4, origin xyz=0.0 0.0 0.0 rpy=0.0 0.0 0.0, axis 1.0 0.0 0.0, limit lower=0.0 upper=0.5 effort=10000 velocity=1
- added joint prismatic_joint_5: type prismatic, parent virtual_link_4, child link_5, origin xyz=0.0 0.0 0.0 rpy=0.0 0.0 0.0, axis 1.0 0.0 0.0, limit lower=0.0 upper=0.5 effort=10000 velocity=1
- added joint revolute_joint_3: type revolute, parent link_2, child virtual_link_2, origin xyz=0.0 0.0 0.0 rpy=0.0 0.0 0.0, axis 0.0 0.0 1.0, limit lower=-0.5236 upper=0.5236 effort=10000 velocity=3
- added joint revolute_joint_4: type revolute, parent link_3, child virtual_link_3, origin xyz=0.0 0.0 0.0 rpy=0.0 0.0 0.0, axis 0.0 0.0 1.0, limit lower=-0.5236 upper=0.5236 effort=10000 velocity=3
- added joint revolute_joint_5: type revolute, parent link_4, child virtual_link_4, origin xyz=0.0 0.0 0.0 rpy=0.0 0.0 0.0, axis 0.0 0.0 1.0, limit lower=-0.5236 upper=0.5236 effort=10000 velocity=3

Commit message: Hackily decrease the mass of each link so that longer robot can still extend

File: assets/urdf/vine.urdf (robot description, URDF)
Before this commit: robot vine_robot, 13 links, 12 joints
Links:
- link base_link: mass 0.1 -> 1
- link link_1: mass 0.1 -> 0.01
- link link_2: mass 0.1 -> 0.001
- link link_3: mass 0.1 -> 0.0001
- link link_4: mass 0.1 -> 0.00001
- link link_5: mass 0.1 -> 0.000001
Joints:
- joint revolute_joint_0: limit lower=-3.146 upper=3.146 effort=10000 velocity=3 -> lower=-0.5236 upper=0.5236 effort=10000 velocity=3
