Commit message: Create fixed base system with parameter and use sparse reward

File: assets/urdf/Vine5LinkFixedBase.urdf (robot description, URDF)
Before this commit: robot vine_robot, 7 links, 6 joints
Joints:
- joint slider_to_cart: axis 0.0 1.0 0.0 -> (none); limit lower=-0.35 upper=0.35 effort=1 velocity=0.5 -> (none); type prismatic -> fixed

Commit message: Remove joint limits to see if the issue goes away

File: assets/urdf/Vine5LinkFixedBase.urdf (robot description, URDF)
Before this commit: robot vine_robot, 7 links, 6 joints
Joints:
- joint cart_to_link_0: limit lower=-0.523599 upper=0.523599 -> (none)
- joint link_0_to_link_1: limit lower=-0.523599 upper=0.523599 -> (none)
- joint link_1_to_link_2: limit lower=-0.523599 upper=0.523599 -> (none)
- joint link_2_to_link_3: limit lower=-0.523599 upper=0.523599 -> (none)
- joint link_3_to_link_4: limit lower=-0.523599 upper=0.523599 -> (none)

Commit message: Trying removing joint limits

File: assets/urdf/Vine5LinkFixedBase.urdf (robot description, URDF)
Before this commit: robot vine_robot, 7 links, 6 joints
Joints:
- joint cart_to_link_0: limit (none) -> lower=-0.523599 upper=0.523599
- joint link_0_to_link_1: limit (none) -> lower=-0.523599 upper=0.523599
- joint link_1_to_link_2: limit (none) -> lower=-0.523599 upper=0.523599
- joint link_2_to_link_3: limit (none) -> lower=-0.523599 upper=0.523599
- joint link_3_to_link_4: limit (none) -> lower=-0.523599 upper=0.523599

File: assets/urdf/Vine5LinkMovingBase.urdf (robot description, URDF)
Before this commit: robot vine_robot, 7 links, 6 joints
Joints:
- joint cart_to_link_0: limit (none) -> lower=-0.523599 upper=0.523599
- joint link_0_to_link_1: limit (none) -> lower=-0.523599 upper=0.523599
- joint link_1_to_link_2: limit (none) -> lower=-0.523599 upper=0.523599
- joint link_2_to_link_3: limit (none) -> lower=-0.523599 upper=0.523599
- joint link_3_to_link_4: limit (none) -> lower=-0.523599 upper=0.523599

Commit message: Remove urdf revolute joint limits

File: assets/urdf/Vine5LinkFixedBase.urdf (robot description, URDF)
Before this commit: robot vine_robot, 7 links, 6 joints
Joints:
- joint cart_to_link_0: limit lower=-0.523599 upper=0.523599 -> (none)
- joint link_0_to_link_1: limit lower=-0.523599 upper=0.523599 -> (none)
- joint link_1_to_link_2: limit lower=-0.523599 upper=0.523599 -> (none)
- joint link_2_to_link_3: limit lower=-0.523599 upper=0.523599 -> (none)
- joint link_3_to_link_4: limit lower=-0.523599 upper=0.523599 -> (none)

File: assets/urdf/Vine5LinkMovingBase.urdf (robot description, URDF)
Before this commit: robot vine_robot, 7 links, 6 joints
Joints:
- joint cart_to_link_0: limit lower=-0.523599 upper=0.523599 -> (none)
- joint link_0_to_link_1: limit lower=-0.523599 upper=0.523599 -> (none)
- joint link_1_to_link_2: limit lower=-0.523599 upper=0.523599 -> (none)
- joint link_2_to_link_3: limit lower=-0.523599 upper=0.523599 -> (none)
- joint link_3_to_link_4: limit lower=-0.523599 upper=0.523599 -> (none)

Commit message: Add tip link because before tip position was actually not at the tip, but at the link before the tip

File: assets/urdf/Vine5LinkFixedBase.urdf (robot description, URDF)
Before this commit: robot vine_robot, 7 links, 6 joints
Links:
- added link tip
Joints:
- added joint link_4_to_tip: type fixed, parent link_4, child tip, origin xyz=0.0 0.0 0.0885 rpy=0.0 0.0 0.0

File: assets/urdf/Vine5LinkMovingBase.urdf (robot description, URDF)
Before this commit: robot vine_robot, 7 links, 6 joints
Links:
- added link tip
Joints:
- added joint link_4_to_tip: type fixed, parent link_4, child tip, origin xyz=0.0 0.0 0.0885 rpy=0.0 0.0 0.0

Commit message: Add cart size bigger in urdf

File: assets/urdf/Vine5LinkFixedBase.urdf (robot description, URDF)
Before this commit: robot vine_robot, 8 links, 7 joints
Links:
- link cart: geometry collision box size=0.07 0.1 0.12; visual box size=0.07 0.1 0.12
Joints:
- joint cart_to_link_0: origin xyz=0.0 0.0 -0.01 rpy=3.1415 0.0 0.0 -> xyz=0.0 0.0 -0.06 rpy=3.1415 0.0 0.0
- joint slider_to_cart: origin xyz=0.0 0.0 -0.025 rpy=0.0 0.0 0.0 -> xyz=0.0 0.0 -0.075 rpy=0.0 0.0 0.0

File: assets/urdf/Vine5LinkMovingBase.urdf (robot description, URDF)
Before this commit: robot vine_robot, 10 links, 9 joints
Links:
- link cart: geometry collision box size=0.07 0.1 0.12; visual box size=0.07 0.1 0.12
Joints:
- joint cart_to_link_0: origin xyz=0.0 0.0 -0.01 rpy=3.1415 0.0 0.0 -> xyz=0.0 0.0 -0.06 rpy=3.1415 0.0 0.0
- joint slider_to_cart: origin xyz=0.0 0.0 -0.025 rpy=0.0 0.0 0.0 -> xyz=0.0 0.0 -0.075 rpy=0.0 0.0 0.0

Commit message: Fix typo from inertia to inertial

File: assets/urdf/Vine5LinkFixedBase.urdf (robot description, URDF)
Before this commit: robot vine_robot, 8 links, 7 joints
Links:
- link cart: mass None -> 0.4

File: assets/urdf/Vine5LinkMovingBase.urdf (robot description, URDF)
Before this commit: robot vine_robot, 10 links, 9 joints
Links:
- link cart: mass None -> 0.4
