Commit message: Update vine urdf to diameter of vine with fpam

File: assets/urdf/Vine5LinkMovingBase_OG.urdf (robot description, URDF)
Before this commit: robot vine_robot, 10 links, 9 joints
Links:
- link link_0: geometry collision cylinder length=0.0885 radius=0.0381; visual cylinder length=0.0885 radius=0.0381
- link link_1: geometry collision cylinder length=0.0885 radius=0.0381; visual cylinder length=0.0885 radius=0.0381
- link link_2: geometry collision cylinder length=0.0885 radius=0.0381; visual cylinder length=0.0885 radius=0.0381
- link link_3: geometry collision cylinder length=0.0885 radius=0.0381; visual cylinder length=0.0885 radius=0.0381
- link link_4: geometry collision cylinder length=0.0885 radius=0.0381; visual cylinder length=0.0885 radius=0.0381
