Commit message: Add contact force penalty, lengthen vine
Co-authored-by: Rianna Jitosho <rjitosho@users.noreply.github.com>

File: assets/urdf/Vine5LinkMovingBase_0885.urdf (robot description, URDF)
Before this commit: robot vine_robot, 8 links, 7 joints
Links:
- link link_0: geometry collision cylinder length=0.0885 radius=0.0169; collision cylinder length=0.0885 radius=0.0381
- link link_1: geometry collision cylinder length=0.0885 radius=0.0169; collision cylinder length=0.0885 radius=0.0381
- link link_2: geometry collision cylinder length=0.0885 radius=0.0169; collision cylinder length=0.0885 radius=0.0381
- link link_3: geometry collision cylinder length=0.0885 radius=0.0169; collision cylinder length=0.0885 radius=0.0381
- link link_4: geometry collision cylinder length=0.0885 radius=0.0169; collision cylinder length=0.0885 radius=0.0381
Joints:
- joint link_0_to_link_1: origin xyz=0.0 0.0 0.0950 rpy=0.0 0.0 0.0 -> xyz=0.0 0.0 0.0885 rpy=0.0 0.0 0.0
- joint link_1_to_link_2: origin xyz=0.0 0.0 0.0950 rpy=0.0 0.0 0.0 -> xyz=0.0 0.0 0.0885 rpy=0.0 0.0 0.0
- joint link_2_to_link_3: origin xyz=0.0 0.0 0.0950 rpy=0.0 0.0 0.0 -> xyz=0.0 0.0 0.0885 rpy=0.0 0.0 0.0
- joint link_3_to_link_4: origin xyz=0.0 0.0 0.0950 rpy=0.0 0.0 0.0 -> xyz=0.0 0.0 0.0885 rpy=0.0 0.0 0.0
- joint link_4_to_tip: origin xyz=0.0 0.0 0.0950 rpy=0.0 0.0 0.0 -> xyz=0.0 0.0 0.0885 rpy=0.0 0.0 0.0
