Commit message: Add rough Vine5LinkMovingBase.urdf

File: assets/urdf/Vine5LinkMovingBase.urdf (robot description, URDF)
Before this commit: robot vine_robot, 0 links, 0 joints
Links:
- added link cart; collision box size=0.2 0.25 0.2; visual box size=0.2 0.25 0.2
- added link link_0, mass 0.0885; collision cylinder length=0.0885 radius=0.015; visual cylinder length=0.0885 radius=0.015
- added link link_1, mass 0.0885; collision cylinder length=0.0885 radius=0.015; visual cylinder length=0.0885 radius=0.015
- added link link_2, mass 0.0885; collision cylinder length=0.0885 radius=0.015; visual cylinder length=0.0885 radius=0.015
- added link link_3, mass 0.0885; collision cylinder length=0.0885 radius=0.015; visual cylinder length=0.0885 radius=0.015
- added link link_4, mass 0.0885; collision cylinder length=0.0885 radius=0.015; visual cylinder length=0.0885 radius=0.015
- added link link_5, mass 0.0885; collision cylinder length=0.0885 radius=0.015; visual cylinder length=0.0885 radius=0.015
- added link slider; collision box size=0.03 8 0.03; visual box size=0.03 8 0.03
Joints:
- added joint cart_to_link_0: type revolute, parent cart, child link_0, origin xyz=0.0 0.0 -0.1 rpy=3.1415 0.0 0.0, axis 1.0 0.0 0.0, limit lower=-0.52 upper=0.52 effort=10000 velocity=8
- added joint link_0_to_link_1: type revolute, parent link_0, child link_1, origin xyz=0.0 0.0 0.0885 rpy=0.0 0.0 0.0, axis 1.0 0.0 0.0, limit lower=-0.52 upper=0.52 effort=10000 velocity=8
- added joint link_1_to_link_2: type revolute, parent link_1, child link_2, origin xyz=0.0 0.0 0.0885 rpy=0.0 0.0 0.0, axis 1.0 0.0 0.0, limit lower=-0.52 upper=0.52 effort=10000 velocity=8
- added joint link_2_to_link_3: type revolute, parent link_2, child link_3, origin xyz=0.0 0.0 0.0885 rpy=0.0 0.0 0.0, axis 1.0 0.0 0.0, limit lower=-0.52 upper=0.52 effort=10000 velocity=8
- added joint link_3_to_link_4: type revolute, parent link_3, child link_4, origin xyz=0.0 0.0 0.0885 rpy=0.0 0.0 0.0, axis 1.0 0.0 0.0, limit lower=-0.52 upper=0.52 effort=10000 velocity=8
- added joint link_4_to_link_5: type revolute, parent link_4, child link_5, origin xyz=0.0 0.0 0.0885 rpy=0.0 0.0 0.0, axis 1.0 0.0 0.0, limit lower=-0.52 upper=0.52 effort=10000 velocity=8
- added joint slider_to_cart: type prismatic, parent slider, child cart, origin xyz=0.0 0.0 0.0 rpy=0.0 0.0 0.0, axis 0.0 1.0 0.0, limit lower=-4.0 upper=4.0 effort=10000 velocity=8

Commit message: Tweak urdf and add randomization in dof init and target

File: assets/urdf/Vine5LinkMovingBase.urdf (robot description, URDF)
Before this commit: robot vine_robot, 8 links, 7 joints
Links:
- link link_0: mass 0.0885 -> 0.005; geometry collision cylinder length=0.0885 radius=0.05; visual cylinder length=0.0885 radius=0.05
- link link_1: mass 0.0885 -> 0.005; geometry collision cylinder length=0.0885 radius=0.05; visual cylinder length=0.0885 radius=0.05
- link link_2: mass 0.0885 -> 0.005; geometry collision cylinder length=0.0885 radius=0.05; visual cylinder length=0.0885 radius=0.05
- link link_3: mass 0.0885 -> 0.005; geometry collision cylinder length=0.0885 radius=0.05; visual cylinder length=0.0885 radius=0.05
- link link_4: mass 0.0885 -> 0.005; geometry collision cylinder length=0.0885 radius=0.05; visual cylinder length=0.0885 radius=0.05
- link link_5: mass 0.0885 -> 0.1; geometry collision cylinder length=0.0885 radius=0.05; visual cylinder length=0.0885 radius=0.05

Commit message: In progress updating urdf file to have 5 links not 6

File: assets/urdf/Vine5LinkMovingBase.urdf (robot description, URDF)
Before this commit: robot vine_robot, 8 links, 7 joints
Links:
- removed link link_5
- link cart: geometry collision box size=0.07 0.1 0.02; visual box size=0.07 0.1 0.02
- link link_0: geometry collision cylinder length=0.0885 radius=0.0381; visual cylinder length=0.0885 radius=0.0381
- link link_1: geometry collision cylinder length=0.0885 radius=0.0381; visual cylinder length=0.0885 radius=0.0381
- link link_2: geometry collision cylinder length=0.0885 radius=0.0381; visual cylinder length=0.0885 radius=0.0381
- link link_3: geometry collision cylinder length=0.0885 radius=0.0381; visual cylinder length=0.0885 radius=0.0381
- link link_4: mass 0.005 -> 0.1; geometry collision cylinder length=0.0885 radius=0.0381; visual cylinder length=0.0885 radius=0.0381
- link slider: geometry collision box size=0.03 8 0.03; visual box size=0.03 0.8 0.03
Joints:
- removed joint link_4_to_link_5
- joint cart_to_link_0: limit lower=-0.52 upper=0.52 effort=10000 velocity=8 -> lower=-0.523599 upper=0.523599; origin xyz=0.0 0.0 -0.1 rpy=3.1415 0.0 0.0 -> xyz=0.0 0.0 -0.01 rpy=3.1415 0.0 0.0
- joint link_0_to_link_1: limit lower=-0.52 upper=0.52 effort=10000 velocity=8 -> lower=-0.523599 upper=0.523599
- joint link_1_to_link_2: limit lower=-0.52 upper=0.52 effort=10000 velocity=8 -> lower=-0.523599 upper=0.523599
- joint link_2_to_link_3: limit lower=-0.52 upper=0.52 effort=10000 velocity=8 -> lower=-0.523599 upper=0.523599
- joint link_3_to_link_4: limit lower=-0.52 upper=0.52 effort=10000 velocity=8 -> lower=-0.523599 upper=0.523599
- joint slider_to_cart: limit lower=-4.0 upper=4.0 effort=10000 velocity=8 -> lower=-0.4 upper=0.4 effort=1 velocity=0.5; origin xyz=0.0 0.0 0.0 rpy=0.0 0.0 0.0 -> xyz=0.0 0.0 -0.025 rpy=0.0 0.0 0.0

Commit message: Adjust urdf joint limits

File: assets/urdf/Vine5LinkMovingBase.urdf (robot description, URDF)
Before this commit: robot vine_robot, 7 links, 6 joints
Joints:
- joint slider_to_cart: limit lower=-0.4 upper=0.4 effort=1 velocity=0.5 -> lower=-0.35 upper=0.35 effort=1 velocity=0.5

Commit message: Play around with no rail system

File: assets/urdf/Vine5LinkMovingBase.urdf (robot description, URDF)
Before this commit: robot vine_robot, 7 links, 6 joints
Joints:
- joint slider_to_cart: limit lower=-0.35 upper=0.35 effort=1 velocity=0.5 -> lower=-0.05 upper=0.05

Commit message: Add experimental changes

File: assets/urdf/Vine5LinkMovingBase.urdf (robot description, URDF)
Before this commit: robot vine_robot, 7 links, 6 joints
Joints:
- joint cart_to_link_0: limit lower=-0.523599 upper=0.523599 -> lower=-1.0 upper=1.0
- joint link_0_to_link_1: limit lower=-0.523599 upper=0.523599 -> lower=-1.0 upper=1.0
- joint link_1_to_link_2: limit lower=-0.523599 upper=0.523599 -> lower=-1.0 upper=1.0
- joint link_2_to_link_3: limit lower=-0.523599 upper=0.523599 -> lower=-1.0 upper=1.0
- joint link_3_to_link_4: limit lower=-0.523599 upper=0.523599 -> lower=-1.0 upper=1.0
- joint slider_to_cart: axis 0.0 1.0 0.0 -> (none); limit lower=-0.05 upper=0.05 -> (none); type prismatic -> fixed

Commit message: Convert from rail force action to rail velocity action, log these, remove joint limits

File: assets/urdf/Vine5LinkMovingBase.urdf (robot description, URDF)
Before this commit: robot vine_robot, 7 links, 6 joints
Joints:
- joint slider_to_cart: limit lower=-0.35 upper=0.35 effort=1 velocity=0.5 -> (none)

Commit message: Add visual limits

File: assets/urdf/Vine5LinkMovingBase.urdf (robot description, URDF)
Before this commit: robot vine_robot, 8 links, 7 joints
Links:
- added link left_limit; visual box size=0.03 0.03 0.2
- added link right_limit; visual box size=0.03 0.03 0.2
Joints:
- added joint slider_to_left_limit: type fixed, parent slider, child left_limit, origin xyz=0.0 -0.2 0.0 rpy=0.0 0.0 0.0
- added joint slider_to_right_limit: type fixed, parent slider, child right_limit, origin xyz=0.0 0.2 0.0 rpy=0.0 0.0 0.0

Commit message: Test 10: Vel reward only

File: assets/urdf/Vine5LinkMovingBase.urdf (robot description, URDF)
Before this commit: robot vine_robot, 10 links, 9 joints
Joints:
- joint slider_to_left_limit: origin xyz=0.0 -0.2 0.0 rpy=0.0 0.0 0.0 -> xyz=0.0 -0.15 0.0 rpy=0.0 0.0 0.0
- joint slider_to_right_limit: origin xyz=0.0 0.2 0.0 rpy=0.0 0.0 0.0 -> xyz=0.0 0.15 0.0 rpy=0.0 0.0 0.0

Commit message: Move pipe to target pos in fixed angle

File: assets/urdf/Vine5LinkMovingBase.urdf (robot description, URDF)
Before this commit: robot vine_robot, 10 links, 9 joints
Joints:
- joint slider_to_left_limit: origin xyz=0.0 -0.15 0.0 rpy=0.0 0.0 0.0 -> xyz=0.0 -0.2 0.0 rpy=0.0 0.0 0.0
- joint slider_to_right_limit: origin xyz=0.0 0.15 0.0 rpy=0.0 0.0 0.0 -> xyz=0.0 0.2 0.0 rpy=0.0 0.0 0.0

Commit message: add many things like net contact force, draw episode line, tune params, sphere size of success dist, widen success dist, widen soft limits, etc.

File: assets/urdf/Vine5LinkMovingBase.urdf (robot description, URDF)
Before this commit: robot vine_robot, 10 links, 9 joints
Joints:
- joint slider_to_left_limit: origin xyz=0.0 -0.2 0.0 rpy=0.0 0.0 0.0 -> xyz=0.0 -0.3 0.0 rpy=0.0 0.0 0.0
- joint slider_to_right_limit: origin xyz=0.0 0.2 0.0 rpy=0.0 0.0 0.0 -> xyz=0.0 0.3 0.0 rpy=0.0 0.0 0.0

Commit message: Add fpam visuals and last collision cylinder (if all, will not be able to bend

File: assets/urdf/Vine5LinkMovingBase.urdf (robot description, URDF)
Before this commit: robot vine_robot, 10 links, 9 joints
Links:
- added link fpam_0; visual cylinder length=0.0885 radius=0.0169
- added link fpam_1; visual cylinder length=0.0885 radius=0.0169
- added link fpam_2; visual cylinder length=0.0885 radius=0.0169
- added link fpam_3; visual cylinder length=0.0885 radius=0.0169
- added link fpam_4; collision cylinder length=0.0885 radius=0.0169; visual cylinder length=0.0885 radius=0.0169
- link link_0: geometry collision cylinder length=0.0885 radius=0.0381; visual cylinder length=0.0885 radius=0.0381
- link link_1: geometry collision cylinder length=0.0885 radius=0.0381; visual cylinder length=0.0885 radius=0.0381
- link link_2: geometry collision cylinder length=0.0885 radius=0.0381; visual cylinder length=0.0885 radius=0.0381
- link link_3: geometry collision cylinder length=0.0885 radius=0.0381; visual cylinder length=0.0885 radius=0.0381
- link link_4: geometry collision cylinder length=0.0885 radius=0.0381; visual cylinder length=0.0885 radius=0.0381
Joints:
- added joint link_0_to_fpam_0: type fixed, parent link_0, child fpam_0, origin xyz=0.0 0.055 0.0 rpy=0.0 0.0 0.0
- added joint link_1_to_fpam_1: type fixed, parent link_1, child fpam_1, origin xyz=0.0 0.055 0.0 rpy=0.0 0.0 0.0
- added joint link_2_to_fpam_2: type fixed, parent link_2, child fpam_2, origin xyz=0.0 0.055 0.0 rpy=0.0 0.0 0.0
- added joint link_3_to_fpam_3: type fixed, parent link_3, child fpam_3, origin xyz=0.0 0.055 0.0 rpy=0.0 0.0 0.0
- added joint link_4_to_fpam_4: type fixed, parent link_4, child fpam_4, origin xyz=0.0 0.055 0.0 rpy=0.0 0.0 0.0

Commit message: Improve collisions for vine fpam in urdf

File: assets/urdf/Vine5LinkMovingBase.urdf (robot description, URDF)
Before this commit: robot vine_robot, 15 links, 14 joints
Links:
- removed link fpam_0
- removed link fpam_1
- removed link fpam_2
- removed link fpam_3
- removed link fpam_4
- link link_0: geometry collision cylinder length=0.0885 radius=0.0169; collision cylinder length=0.0885 radius=0.0381
- link link_1: geometry collision cylinder length=0.0885 radius=0.0169; collision cylinder length=0.0885 radius=0.0381
- link link_2: geometry collision cylinder length=0.0885 radius=0.0169; collision cylinder length=0.0885 radius=0.0381
- link link_3: geometry collision cylinder length=0.0885 radius=0.0169; collision cylinder length=0.0885 radius=0.0381
- link link_4: geometry collision cylinder length=0.0885 radius=0.0169; collision cylinder length=0.0885 radius=0.0381
Joints:
- removed joint link_0_to_fpam_0
- removed joint link_1_to_fpam_1
- removed joint link_2_to_fpam_2
- removed joint link_3_to_fpam_3
- removed joint link_4_to_fpam_4

Commit message: Draw rail soft limits with lines instead of urdf to be less brittle

File: assets/urdf/Vine5LinkMovingBase.urdf (robot description, URDF)
Before this commit: robot vine_robot, 10 links, 9 joints
Links:
- removed link left_limit
- removed link right_limit
Joints:
- removed joint slider_to_left_limit
- removed joint slider_to_right_limit

Commit message: Update urdf to have cleaner vine link lengths

File: assets/urdf/Vine5LinkMovingBase.urdf (robot description, URDF)
Before this commit: robot vine_robot, 8 links, 7 joints
Links:
- link link_0: geometry collision cylinder length=0.1 radius=0.0169; collision cylinder length=0.1 radius=0.0381
- link link_1: geometry collision cylinder length=0.0885 radius=0.0169; collision cylinder length=0.0885 radius=0.0381
- link link_2: geometry collision cylinder length=0.0885 radius=0.0169; collision cylinder length=0.0885 radius=0.0381
- link link_3: geometry collision cylinder length=0.0885 radius=0.0169; collision cylinder length=0.0885 radius=0.0381
- link link_4: geometry collision cylinder length=0.0885 radius=0.0169; collision cylinder length=0.0885 radius=0.0381
Joints:
- joint link_0_to_link_1: origin xyz=0.0 0.0 0.0950 rpy=0.0 0.0 0.0 -> xyz=0.0 0.0 0.0885 rpy=0.0 0.0 0.0
- joint link_1_to_link_2: origin xyz=0.0 0.0 0.0950 rpy=0.0 0.0 0.0 -> xyz=0.0 0.0 0.0885 rpy=0.0 0.0 0.0
- joint link_2_to_link_3: origin xyz=0.0 0.0 0.0950 rpy=0.0 0.0 0.0 -> xyz=0.0 0.0 0.0885 rpy=0.0 0.0 0.0
- joint link_3_to_link_4: origin xyz=0.0 0.0 0.0950 rpy=0.0 0.0 0.0 -> xyz=0.0 0.0 0.0885 rpy=0.0 0.0 0.0
- joint link_4_to_tip: origin xyz=0.0 0.0 0.0950 rpy=0.0 0.0 0.0 -> xyz=0.0 0.0 0.0885 rpy=0.0 0.0 0.0

Commit message: Udpate vine urdf
Co-authored-by: Rianna Jitosho <rjitosho@users.noreply.github.com>

File: assets/urdf/Vine5LinkMovingBase.urdf (robot description, URDF)
Before this commit: robot vine_robot, 8 links, 7 joints
Joints:
- joint link_0_to_link_1: origin xyz=0.0 0.0 0.0885 rpy=0.0 0.0 0.0 -> xyz=0.0 0.0 0.1000 rpy=0.0 0.0 0.0

Commit message: Save progress, pretty good but need white squares

File: assets/urdf/Vine5LinkMovingBase.urdf (robot description, URDF)
Before this commit: robot vine_robot, 8 links, 7 joints
Links:
- added link connector, mass 0.0; collision box size=0.08 0.08 0.09; visual box size=0.08 0.08 0.09
Joints:
- removed joint cart_to_link_0
- added joint cart_to_connector: type fixed, parent cart, child connector, origin xyz=0.0 0.0 -0.055 rpy=0.0 0.0 0.0
- added joint connector_to_link_0: type revolute, parent connector, child link_0, origin xyz=0.0 0.0 -0.045 rpy=3.1415 0.0 0.0, axis 1.0 0.0 0.0

Commit message: Add mocap squares

File: assets/urdf/Vine5LinkMovingBase.urdf (robot description, URDF)
Before this commit: robot vine_robot, 9 links, 8 joints
Links:
- added link mocap_square_0; collision box size=0.0005 0.045 0.045; visual box size=0.0005 0.045 0.045
- added link mocap_square_1; collision box size=0.0005 0.045 0.045; visual box size=0.0005 0.045 0.045
- added link mocap_square_2; collision box size=0.0005 0.045 0.045; visual box size=0.0005 0.045 0.045
- added link mocap_square_3; collision box size=0.0005 0.045 0.045; visual box size=0.0005 0.045 0.045
- added link mocap_square_4; collision box size=0.0005 0.045 0.045; visual box size=0.0005 0.045 0.045
Joints:
- added joint link_0_to_mocap_square_0: type fixed, parent link_0, child mocap_square_0, origin xyz=0.0381 0.0 0.04425 rpy=0.0 0.0 0.0
- added joint link_1_to_mocap_square_1: type fixed, parent link_1, child mocap_square_1, origin xyz=0.0381 0.0 0.04425 rpy=0.0 0.0 0.0
- added joint link_2_to_mocap_square_2: type fixed, parent link_2, child mocap_square_2, origin xyz=0.0381 0.0 0.04425 rpy=0.0 0.0 0.0
- added joint link_3_to_mocap_square_3: type fixed, parent link_3, child mocap_square_3, origin xyz=0.0381 0.0 0.04425 rpy=0.0 0.0 0.0
- added joint link_4_to_mocap_square_4: type fixed, parent link_4, child mocap_square_4, origin xyz=0.0381 0.0 0.04425 rpy=0.0 0.0 0.0

Commit message: Remove collisions of mocap

File: assets/urdf/Vine5LinkMovingBase.urdf (robot description, URDF)
Before this commit: robot vine_robot, 14 links, 13 joints
Links:
- link mocap_square_0: geometry visual box size=0.0005 0.045 0.045
- link mocap_square_1: geometry visual box size=0.0005 0.045 0.045
- link mocap_square_2: geometry visual box size=0.0005 0.045 0.045
- link mocap_square_3: geometry visual box size=0.0005 0.045 0.045
- link mocap_square_4: geometry visual box size=0.0005 0.045 0.045
