Commit message: Add 1 spherical link for 3D model
Co-authored-by: Rianna Jitosho <rjitosho@users.noreply.github.com>

File: assets/urdf/Vine5LinkMovingBase3D.urdf (robot description, URDF)
Before this commit: robot vine_robot, 13 links, 12 joints
Links:
- removed link fake_link_0
- removed link fake_link_1
- removed link fake_link_2
- removed link fake_link_3
- removed link fake_link_4
Joints:
- removed joint cart_to_fake_link_0
- removed joint fake_link_0_to_link_0
- removed joint fake_link_1_to_link_1
- removed joint fake_link_2_to_link_2
- removed joint fake_link_3_to_link_3
- removed joint fake_link_4_to_link_4
- removed joint link_0_to_fake_link_1
- removed joint link_1_to_fake_link_2
- removed joint link_2_to_fake_link_3
- removed joint link_3_to_fake_link_4
- added joint cart_to_link_0: type spherical, parent cart, child link_0, origin xyz=0.0 0.0 -0.01 rpy=3.1415 0.0 0.0, axis 1.0 0.0 0.0
- added joint link_0_to_link_1: type revolute, parent link_0, child link_1, origin xyz=0.0 0.0 0.0885 rpy=0.0 0.0 0.0, axis 1.0 0.0 0.0
- added joint link_1_to_link_2: type revolute, parent link_1, child link_2, origin xyz=0.0 0.0 0.0885 rpy=0.0 0.0 0.0, axis 1.0 0.0 0.0
- added joint link_2_to_link_3: type revolute, parent link_2, child link_3, origin xyz=0.0 0.0 0.0885 rpy=0.0 0.0 0.0, axis 1.0 0.0 0.0
- added joint link_3_to_link_4: type revolute, parent link_3, child link_4, origin xyz=0.0 0.0 0.0885 rpy=0.0 0.0 0.0, axis 1.0 0.0 0.0

Commit message: Switch to 2 revolute joints for 3D motion
Co-authored-by: Rianna Jitosho <rjitosho@users.noreply.github.com>

File: assets/urdf/Vine5LinkMovingBase3D.urdf (robot description, URDF)
Before this commit: robot vine_robot, 8 links, 7 joints
Links:
- added link rotation_y
Joints:
- removed joint cart_to_link_0
- added joint cart_to_rotation_y: type revolute, parent cart, child rotation_y, origin xyz=0.0 0.0 -0.01 rpy=3.1415 0.0 0.0, axis 1.0 0.0 0.0
- added joint rotation_y_to_link_0: type revolute, parent rotation_y, child link_0, origin xyz=0.0 0.0 0.0 rpy=0.0 0.0 0.0, axis 0.0 1.0 0.0

Commit message: Fix collision filter, works with KCBb

File: assets/urdf/Vine5LinkMovingBase3D.urdf (robot description, URDF)
Before this commit: robot vine_robot, 9 links, 8 joints
Joints:
- joint cart_to_rotation_y: axis 1.0 0.0 0.0 -> 0.0 1.0 0.0; origin xyz=0.0 0.0 -0.01 rpy=3.1415 0.0 0.0 -> xyz=0.0 0.0 -0.015 rpy=3.1415 0.0 0.0
- joint rotation_y_to_link_0: axis 0.0 1.0 0.0 -> 1.0 0.0 0.0

Commit message: Add prismatic joint to 3D model
Co-authored-by: Rianna Jitosho <rjitosho@users.noreply.github.com>

File: assets/urdf/Vine5LinkMovingBase3D.urdf (robot description, URDF)
Before this commit: robot vine_robot, 9 links, 8 joints
Links:
- added link translation_z
Joints:
- removed joint cart_to_rotation_y
- added joint cart_to_translation_z: type prismatic, parent cart, child translation_z, origin xyz=0.0 0.0 -0.015 rpy=3.1415 0.0 0.0, axis 0.0 0.0 1.0, limit lower=-0.35 upper=0.35 effort=1 velocity=0.5
- added joint translation_z_to_rotation_y: type revolute, parent translation_z, child rotation_y, origin xyz=0.0 0.0 0.0 rpy=0.0 0.0 0.0, axis 0.0 1.0 0.0

Commit message: Add growth RL action

File: assets/urdf/Vine5LinkMovingBase3D.urdf (robot description, URDF)
Before this commit: robot vine_robot, 10 links, 9 joints
Joints:
- joint cart_to_translation_z: limit lower=-0.35 upper=0.35 effort=1 velocity=0.5 -> lower=0 upper=0.35 effort=1 velocity=0.05

Commit message: Rotate vine 90 degrees

File: assets/urdf/Vine5LinkMovingBase3D.urdf (robot description, URDF)
Before this commit: robot vine_robot, 10 links, 9 joints
Joints:
- joint translation_z_to_rotation_y: origin xyz=0.0 0.0 0.0 rpy=0.0 0.0 0.0 -> xyz=0.0 0.0 0.0 rpy=0.0 0.0 -1.5708

Commit message: Swap order of translation_z and rotation_y

File: assets/urdf/Vine5LinkMovingBase3D.urdf (robot description, URDF)
Before this commit: robot vine_robot, 10 links, 9 joints
Joints:
- removed joint cart_to_translation_z
- removed joint rotation_y_to_link_0
- removed joint translation_z_to_rotation_y
- added joint cart_to_rotation_y: type revolute, parent cart, child rotation_y, origin xyz=0.0 0.0 -0.015 rpy=3.1415 0.0 1.5708, axis 0.0 1.0 0.0
- added joint rotation_y_to_translation_z: type prismatic, parent rotation_y, child translation_z, origin xyz=0.0 0.0 0.0 rpy=0.0 0.0 0.0, axis 0.0 0.0 1.0, limit lower=0 upper=0.35 effort=1 velocity=0.05
- added joint translation_z_to_link_0: type revolute, parent translation_z, child link_0, origin xyz=0.0 0.0 0.0 rpy=0.0 0.0 0.0, axis 1.0 0.0 0.0
