Commit message: Modify urdf files to point to relative paths to meshes and remove gazebo tags

File: assets/urdf/shelf/urdf/shelf.urdf (robot description, URDF)
Before this commit: robot shelf, 1 links, 0 joints
Links:
- link base_link: geometry collision mesh filename=../meshes/shelf.stl; visual mesh filename=../meshes/shelf.stl

File: assets/urdf/shelf_super_market1/urdf/shelf_super_market1.urdf (robot description, URDF)
Before this commit: robot shelf_super_market1, 1 links, 0 joints
Links:
- link base_link: geometry collision mesh filename=../meshes/shelf_super_market1.dae scale=1 1 1; visual mesh filename=../meshes/shelf_super_market1.dae scale=1 1 1

File: assets/urdf/shelf_super_market2/urdf/shelf_super_market2.urdf (robot description, URDF)
Before this commit: robot shelf_super_market2, 1 links, 0 joints
Links:
- link base_link: geometry collision mesh filename=../meshes/shelf_super_market2.dae scale=1 1 1; visual mesh filename=../meshes/shelf_super_market2.dae scale=1 1 1

File: assets/urdf/sushi_shelf/urdf/sushi_shelf.urdf (robot description, URDF)
Before this commit: robot sushi_shelf_model, 1 links, 0 joints
Links:
- link sushi_shelf: geometry collision mesh filename=../meshes/sushi_shelf.dae scale=1.0 1.0 1.0; visual mesh filename=../meshes/sushi_shelf.dae scale=1.0 1.0 1.0

Commit message: Try switching to .obj instead of .stl (still doesn't work)

File: assets/urdf/shelf/urdf/shelf.urdf (robot description, URDF)
Before this commit: robot shelf, 1 links, 0 joints
Links:
- link base_link: geometry collision mesh filename=../meshes/shelf.obj; visual mesh filename=../meshes/shelf.obj
