Commit message: Update shelf color and geometry, move z targets higher

File: assets/urdf/shelf/urdf/custom_shelf_old.urdf (robot description, URDF)
Before this commit: robot shelf, 1 links, 0 joints
Links:
- link shelf: geometry collision box size=0.025 0.025 0.75; collision box size=0.025 0.025 0.75
