Commit message: Fix collision issue skipping between control steps

File: assets/urdf/shelf/urdf/custom_shelf.urdf (robot description, URDF)
Before this commit: robot shelf, 1 links, 0 joints
Links:
- removed link shelf
- added link shelf_link, mass 500; collision box size=0.025 0.025 0.75; collision box size=0.025 0.025 0.75

Commit message: Update shelf for penalty only on side
Co-authored-by: Rianna Jitosho <rjitosho@users.noreply.github.com>

File: assets/urdf/shelf/urdf/custom_shelf.urdf (robot description, URDF)
Before this commit: robot shelf, 1 links, 0 joints
Links:
- added link main_surface; collision box size=0.15 0.399 0.011; visual box size=0.15 0.399 0.011
- link shelf_link: geometry collision box size=0.15 0.4 0.01; collision box size=0.15 0.4 0.01
Joints:
- added joint surface_to_shelf: type fixed, parent shelf_link, child main_surface, origin xyz=0.0 0.0 0.0 rpy=0.0 0.0 0.0, axis 0.0 0.0 0.0

Commit message: Improve shelf urdf for side penalty
Co-authored-by: Rianna Jitosho <rjitosho@users.noreply.github.com>

File: assets/urdf/shelf/urdf/custom_shelf.urdf (robot description, URDF)
Before this commit: robot shelf, 2 links, 1 joints
Links:
- removed link main_surface
- added link shelf, mass 500; collision box size=0.15 0.399 0.01; collision box size=0.15 0.4 0.01
- link shelf_link: mass 500 -> None; geometry collision box size=0.15 0.002 0.01; visual box size=0.15 0.002 0.01
Joints:
- joint surface_to_shelf: child main_surface -> shelf_link; parent shelf_link -> shelf
