Commit message: Increase mesh resolution, add visual check for pipe

File: assets/urdf/pipe/urdf/pipe.urdf (robot description, URDF)
Before this commit: robot pipe, 1 links, 0 joints
Links:
- link base_link: geometry collision mesh filename=../meshes/cylinder-13_8cm-ID.STL; visual mesh filename=../meshes/cylinder-13_8cm-ID.STL
